Commit message: added inertial control to URDF & ran the Rviz2 sim

File: description/robot_core.xacro (robot description, xacro)
@@ -1,4 +1,5 @@
 <?xml version="1.0"?>
 <robot xmlns:xacro="http://www.ros.org/wiki/xacro">
+    <xacro:include filename="inertial_macros.xacro" />
     <material name="white">
         <color rgba="1 1 1 1 "/>
@@ -36,4 +37,7 @@
             </geometry>
         </collision>
+        <xacro: inertial_box mass="0.5" x="0.3" y="0.3" z="0.15">
+            <origin xyz="0.15 0 0.075" rpy="0 0 0"/>
+        </xacro:inertial_box>
     </link>
     <!--  left wheel -->
@@ -56,4 +60,7 @@
         </geometry>
         </collision>
+        <xacro:inertial_cylinder mass="0.1" lenght="0.04" radius="0.05">
+            <origin xyz="0 0 0" rpy="0 0 0"/>
+        </xacro:inertial_cylinder>
     </link>
     <!--  right wheel -->
@@ -76,4 +83,7 @@
         </geometry>
         </collision>
+        <xacro:inertial_cylinder mass="0.1" lenght="0.04" radius="0.05">
+            <origin xyz="0 0 0" rpy="0 0 0"/>
+        </xacro:inertial_cylinder>
     </link>
     <!-- caster wheel-->
@@ -95,4 +105,7 @@
         </geometry>
         </collision>
+        <xacro:inertial_sphere mass="0.1" radius="0.05">
+            <origin xyz="0 0 0" rpy="0 0 0"/>
+        <xacro:inertial_sphere>
     </link>
 </robot>

Commit message: added Gazebo sim and Gazebo controls4

File: description/robot_core.xacro (robot description, xacro)
@@ -37,8 +37,11 @@
             </geometry>
         </collision>
-        <xacro: inertial_box mass="0.5" x="0.3" y="0.3" z="0.15">
+        <xacro:inertial_box mass="0.5" x="0.3" y="0.3" z="0.15">
             <origin xyz="0.15 0 0.075" rpy="0 0 0"/>
         </xacro:inertial_box>
     </link>
+    <gazebo reference="chassis">
+        <material>Gazebo/White</material>
+    </gazebo>
     <!--  left wheel -->
     <joint name="left_wheel_joint" type="continuous">
@@ -60,8 +63,11 @@
         </geometry>
         </collision>
-        <xacro:inertial_cylinder mass="0.1" lenght="0.04" radius="0.05">
+        <xacro:inertial_cylinder mass="0.1" length="0.04" radius="0.05">
             <origin xyz="0 0 0" rpy="0 0 0"/>
         </xacro:inertial_cylinder>
     </link>
+    <gazebo reference="left_wheel">
+        <material>Gazebo/Blue</material>
+    </gazebo>
     <!--  right wheel -->
     <joint name="right_wheel_joint" type="continuous">
@@ -83,8 +89,11 @@
         </geometry>
         </collision>
-        <xacro:inertial_cylinder mass="0.1" lenght="0.04" radius="0.05">
+        <xacro:inertial_cylinder mass="0.1" length="0.04" radius="0.05">
             <origin xyz="0 0 0" rpy="0 0 0"/>
         </xacro:inertial_cylinder>
     </link>
+    <gazebo reference="right_wheel">
+        <material>Gazebo/Blue</material>
+    </gazebo>
     <!-- caster wheel-->
     <joint name="caster_wheel_joint" type="fixed">
@@ -107,5 +116,8 @@
         <xacro:inertial_sphere mass="0.1" radius="0.05">
             <origin xyz="0 0 0" rpy="0 0 0"/>
-        <xacro:inertial_sphere>
+        </xacro:inertial_sphere>
     </link>
+    <gazebo reference="caster_wheel">
+        <material>Gazebo/Black</material>
+    </gazebo>
 </robot>
